File: electrical/USB-PD-Breakout.sch (KiCad schematic (older format))
At the start: 15 parts, among them J1 USB-C_Female, J2 CONN_02X04, J3 USB_A, J4 CONN_01X05, J5 CONN_01X02, U1 FUSB302MPX

Commit message: Rev2 Update
Parts:
- removed J2: CONN_02X04, Socket_Strips:Socket_Strip_Straight_2x04, symbol CONN_02X04
- removed J3: USB_A, Jason_Libraries:USB_A_Female_SMD, symbol USB_A
- removed J4: CONN_01X05, Socket_Strips:Socket_Strip_Straight_1x05, symbol CONN_01X05
- removed J5: CONN_01X02, Socket_Strips:Socket_Strip_Straight_1x02, symbol CONN_01X02
- added J2: USB_OTG, Reclaimer_Labs:USB_Micro-B_10118193, symbol USB_OTG-RESCUE-USB-PD-Breakout
- added J3, J4, J5: CONN_02X03, Socket_Strips:Socket_Strip_Straight_2x03, symbol CONN_02X03
- added X1, X2, X3, X4: MTHOLE, Reclaimer_Labs:MountingHole_3.5mm_Pad_Via, symbol MTHOLE
- C1: value 22uF -> 10uF; footprint Jason_Libraries:R_0805 -> Capacitors_SMD:C_1206; MacroFab Part Number (none) -> MF-CAP-1206-10uF; Manufacturer Yageo -> (none); Manufacturer Part Number CC0805MKX5R6BB226 -> (none); Supplier 1 Digikey -> (none); Supplier 1 Part Number 311-1900-2-ND -> (none)
- C2, C4: footprint Jason_Libraries:0603_np -> Capacitors_SMD:C_0603; MacroFab Part Number (none) -> MF-CAP-0603-0.1uF; Manufacturer Yageo -> (none); Manufacturer Part Number CC0603KRX7R7BB104 -> (none); Supplier 1 Digikey -> (none); Supplier 1 Part Number 311-1088-1-ND -> (none)
- C3: footprint Jason_Libraries:R_0805 -> Capacitors_SMD:C_0805; MacroFab Part Number (none) -> MF-CAP-0805-1uF; Manufacturer Yageo -> (none); Manufacturer Part Number CC0805KKX7R7BB105 -> (none); Supplier 1 Digikey -> (none); Supplier 1 Part Number 311-1365-1-ND -> (none)
- C5, C6: footprint Jason_Libraries:0603_np -> Capacitors_SMD:C_0603
- J1: footprint Jason_Libraries:USB-C_Female_Top_Mount_Dual_SMT_RA -> Reclaimer_Labs:USB-C_Female_105450-0101; Manufacturer JAE Electronics -> Molex; Manufacturer Part Number DX07S024JJ3R1300 -> 1054500101; Supplier 1 Part Number 670-2846-1-ND -> WM12856CT-ND
- R1: renamed from R2; footprint Jason_Libraries:R_0805 -> Capacitors_SMD:C_0603; MacroFab Part Number (none) -> MF-RES-0603-4.7K
- R2: renamed from R3; footprint Jason_Libraries:R_0805 -> Capacitors_SMD:C_0603; MacroFab Part Number (none) -> MF-RES-0603-4.7K
- R3: renamed from R4; footprint Jason_Libraries:R_0805 -> Capacitors_SMD:C_0603; MacroFab Part Number (none) -> MF-RES-0603-4.7K
- U1: value FUSB302MPX -> FUSB302BMPX; footprint Jason_Libraries:MLP_14 -> Reclaimer_Labs:MLP_14; Manufacturer Part Number FUSB302MPX -> FUSB302BMPX; Supplier 1 Mouser -> Digikey; Supplier 1 Part Number 512-FUSB302MPX -> FUSB302BMPXCT-ND
Connections:
- net labels added: USB20_D+, USB20_D-, USBC_CC1, USBC_CC2, VBUS_A, VBUS_C, VCONN, VDD, V_PULLUP
- net labels removed: CC1, CC2, D+, D-, Vbus, VbusA, Vconn, Vdd, Vpu
- wire segments 72 -> 96
- no-connect marks 10 -> 13
Other:
- note added: "USB 2.0 signals have two possible positions. \nWe connect both together so either plug orientation will work. \nRoute to minimize stub lengths."
- moved on the sheet: C1, C2, C3, C4, C5, C6, J1, R1, R2, R3, U1
